Commit message: LBR iiwa base-flange transform fix
Changed the tool0 and flange joint origin to represent real lrb iiwa 14 flange frame. Fixing issue #72

(cherry picked from commit d8f5c57a34ca6cb18672831b3119c5915ad60eb1)

File: kuka_lbr_iiwa_support/urdf/lbr_iiwa14_r820_macro.xacro (robot description, xacro)
@@ -1,3 +1,3 @@
-<?xml version="1.0"?>
+<?xml version="1.0" encoding="UTF-8"?>
 <robot xmlns:xacro="http://wiki.ros.org/xacro">
   <!-- include helper xacros -->
@@ -11,4 +11,5 @@
         </geometry>
         <origin rpy="-0.0 0.0 0.0" xyz="0.0 0.0 0.0"/>
+        <xacro:material_kuka_ral_gray_aluminium/>
       </visual>
       <collision>
@@ -18,4 +19,9 @@
         </geometry>
       </collision>
+      <inertial>
+        <inertia ixx="1.0" ixy="0.0" ixz="0.0" iyy="1.0" iyz="0.0" izz="1.0"/>
+        <mass value="8.666E0"/>
+        <origin rpy="0.0 0.0 0.0" xyz="0.0 0.0 0.0"/>
+      </inertial>
     </link>
     <link name="${prefix}link_1">
@@ -25,4 +31,5 @@
         </geometry>
         <origin rpy="-0.0 0.0 0.0" xyz="0.0 0.0 0.0"/>
+        <xacro:material_kuka_ral_gray_aluminium/>
       </visual>
       <collision>
@@ -32,4 +39,9 @@
         </geometry>
       </collision>
+      <inertial>
+        <inertia ixx="0.0489108039022503" ixy="0.0" ixz="0.0" iyy="0.0383705935400879" iyz="0.0" izz="0.0522121642769911"/>
+        <mass value="9.62E0"/>
+        <origin rpy="-1.3035636348359196 -0.7815781053554747 1.2529437882898196" xyz="0.00344301039501039 0.0191980353430353 0.08662803846153849"/>
+      </inertial>
     </link>
     <link name="${prefix}link_2">
@@ -39,4 +51,5 @@
         </geometry>
         <origin rpy="-0.0 0.0 0.0" xyz="0.0 0.0 0.0"/>
+        <xacro:material_kuka_orange/>
       </visual>
       <collision>
@@ -46,4 +59,9 @@
         </geometry>
       </collision>
+      <inertial>
+        <inertia ixx="0.0306168627253135" ixy="0.0" ixz="0.0" iyy="0.252047093745431" iyz="0.0" izz="0.258650362609461"/>
+        <mass value="8.079E0"/>
+        <origin rpy="0.017400716172763755 1.2184236596039677E-4 7.609596915052352E-4" xyz="0.144939171927219 4.90834261666048E-4 0.0453728741180839"/>
+      </inertial>
     </link>
     <link name="${prefix}link_3">
@@ -53,4 +71,5 @@
         </geometry>
         <origin rpy="-0.0 0.0 0.0" xyz="0.0 0.0 0.0"/>
+        <xacro:material_kuka_ral_gray_aluminium/>
       </visual>
       <collision>
@@ -60,4 +79,9 @@
         </geometry>
       </collision>
+      <inertial>
+        <inertia ixx="0.0181557035426496" ixy="0.0" ixz="0.0" iyy="0.0346916391676837" iyz="0.0" izz="0.037776951242458"/>
+        <mass value="7.6604E0"/>
+        <origin rpy="0.1692981167548117 0.5271433699021747 -2.9605806714357508" xyz="0.0400709362435382 0.00400998642368544 0.0499127101717926"/>
+      </inertial>
     </link>
     <link name="${prefix}link_4">
@@ -67,4 +91,5 @@
         </geometry>
         <origin rpy="-0.0 0.0 0.0" xyz="0.0 0.0 0.0"/>
+        <xacro:material_kuka_orange/>
       </visual>
       <collision>
@@ -74,4 +99,9 @@
         </geometry>
       </collision>
+      <inertial>
+        <inertia ixx="0.0208771593304277" ixy="0.0" ixz="0.0" iyy="0.0526135698207455" iyz="0.0" izz="0.0587485883681802"/>
+        <mass value="5.7014E0"/>
+        <origin rpy="1.535166999601284 -1.2065715961818437 -1.512863903166617" xyz="0.00141160065948714 0.060839292103693904 -0.12025970463395"/>
+      </inertial>
     </link>
     <link name="${prefix}link_5">
@@ -81,4 +111,5 @@
         </geometry>
         <origin rpy="-0.0 0.0 0.0" xyz="0.0 0.0 0.0"/>
+        <xacro:material_kuka_ral_gray_aluminium/>
       </visual>
       <collision>
@@ -88,4 +119,9 @@
         </geometry>
       </collision>
+      <inertial>
+        <inertia ixx="0.0208771593304277" ixy="0.0" ixz="0.0" iyy="0.0526135698207455" iyz="0.0" izz="0.0587485883681802"/>
+        <mass value="5.7014E0"/>
+        <origin rpy="1.535166999601284 -1.2065715961818437 -1.512863903166617" xyz="0.00141160065948714 0.060839292103693904 -0.12025970463395"/>
+      </inertial>
     </link>
     <link name="${prefix}link_6">
@@ -95,4 +131,5 @@
         </geometry>
         <origin rpy="-0.0 0.0 0.0" xyz="0.0 0.0 0.0"/>
+        <xacro:material_kuka_orange/>
       </visual>
       <collision>
@@ -102,4 +139,9 @@
         </geometry>
       </collision>
+      <inertial>
+        <inertia ixx="0.00390274036654823" ixy="0.0" ixz="0.0" iyy="0.00286930887521153" iyz="0.0" izz="0.00403512413298348"/>
+        <mass value="1.509E0"/>
+        <origin rpy="0.051936335875096745 -0.1296523529795729 0.0038347791577379832" xyz="-5.61365142478463E-4 0.00904387011265739 0.0494449237905898"/>
+      </inertial>
     </link>
     <link name="${prefix}link_7">
@@ -109,4 +151,5 @@
         </geometry>
         <origin rpy="-0.0 0.0 0.0" xyz="0.0 0.0 0.0"/>
+        <xacro:material_kuka_ral_gray_aluminium/>
       </visual>
       <collision>
@@ -116,4 +159,9 @@
         </geometry>
       </collision>
+      <inertial>
+        <inertia ixx="0.00390274036654823" ixy="0.0" ixz="0.0" iyy="0.00286930887521153" iyz="0.0" izz="0.00403512413298348"/>
+        <mass value="1.509E0"/>
+        <origin rpy="0.051936335875096745 -0.1296523529795729 0.0038347791577379832" xyz="-5.61365142478463E-4 0.00904387011265739 0.0494449237905898"/>
+      </inertial>
     </link>
     <!-- joints - main serial chain -->

Commit message: temporary fix for effort limit gz sim
Fixing the issue where the `kuka_gazebo` node with the `lbr_iiwa` description doesn't work as the robot drops on the floor under gravity. The effort limits for each joint where taken from iisy description. Temp fixing #96

(cherry picked from commit 25904f147004e282cff014073690aa70fe00c1f2)

File: kuka_lbr_iiwa_support/urdf/lbr_iiwa14_r820_macro.xacro (robot description, xacro)
@@ -171,5 +171,5 @@
       <origin rpy="-0.0 0.0 0.0" xyz="0.0 0.0 0.1575"/>
       <axis xyz="0.0 0.0 1.0"/>
-      <limit effort="0" lower="${radians(-170)}" upper="${radians(170)}" velocity="${radians(85)}"/>
+      <limit effort="398.011277" lower="${radians(-170)}" upper="${radians(170)}" velocity="${radians(85)}"/>
     </joint>
     <joint name="${prefix}joint_2" type="revolute">
@@ -178,5 +178,5 @@
       <origin rpy="-0.0 0.0 0.0" xyz="0.0 0.0 0.2025"/>
       <axis xyz="0.0 1.0 0.0"/>
-      <limit effort="0" lower="${radians(-120)}" upper="${radians(120)}" velocity="${radians(85)}"/>
+      <limit effort="286.529873" lower="${radians(-120)}" upper="${radians(120)}" velocity="${radians(85)}"/>
     </joint>
     <joint name="${prefix}joint_3" type="revolute">
@@ -185,5 +185,5 @@
       <origin rpy="-0.0 0.0 0.0" xyz="0.0 0.0 0.2045"/>
       <axis xyz="0.0 0.0 1.0"/>
-      <limit effort="0" lower="${radians(-170)}" upper="${radians(170)}" velocity="${radians(100)}"/>
+      <limit effort="286.529873" lower="${radians(-170)}" upper="${radians(170)}" velocity="${radians(100)}"/>
     </joint>
     <joint name="${prefix}joint_4" type="revolute">
@@ -192,5 +192,5 @@
       <origin rpy="-0.0 0.0 0.0" xyz="0.0 0.0 0.2155"/>
       <axis xyz="0.0 -1.0 0.0"/>
-      <limit effort="0" lower="${radians(-120)}" upper="${radians(120)}" velocity="${radians(75)}"/>
+      <limit effort="137.666701" lower="${radians(-120)}" upper="${radians(120)}" velocity="${radians(75)}"/>
     </joint>
     <joint name="${prefix}joint_5" type="revolute">
@@ -199,5 +199,5 @@
       <origin rpy="-0.0 0.0 0.0" xyz="0.0 0.0 0.1845"/>
       <axis xyz="0.0 0.0 1.0"/>
-      <limit effort="0" lower="${radians(-170)}" upper="${radians(170)}" velocity="${radians(130)}"/>
+      <limit effort="63.574238" lower="${radians(-170)}" upper="${radians(170)}" velocity="${radians(130)}"/>
     </joint>
     <joint name="${prefix}joint_6" type="revolute">
@@ -206,5 +206,5 @@
       <origin rpy="-0.0 0.0 0.0" xyz="0.0 0.0 0.2155"/>
       <axis xyz="0.0 1.0 0.0"/>
-      <limit effort="0" lower="${radians(-120)}" upper="${radians(120)}" velocity="${radians(135)}"/>
+      <limit effort="58.580298" lower="${radians(-120)}" upper="${radians(120)}" velocity="${radians(135)}"/>
     </joint>
     <joint name="${prefix}joint_7" type="revolute">
@@ -213,5 +213,5 @@
       <origin rpy="-0.0 0.0 0.0" xyz="0.0 0.0 0.081"/>
       <axis xyz="0.0 0.0 1.0"/>
-      <limit effort="0" lower="${radians(-175)}" upper="${radians(175)}" velocity="${radians(135)}"/>
+      <limit effort="15.927568" lower="${radians(-175)}" upper="${radians(175)}" velocity="${radians(135)}"/>
     </joint>
     <!-- ROS-Industrial 'base' frame - equivalent of 'KUKA ROBROOT'-->
