Commit message: removal of world link and added arg for custom fixed parent link
temp fix to #103 for custom linear positioner case

File: kuka_fortec_support/urdf/kr560_r3100_2_macro.xacro (robot description, xacro)
@@ -1,7 +1,6 @@
 <?xml version="1.0"?>
 <robot xmlns:xacro="http://wiki.ros.org/xacro">
-  <xacro:macro name="kuka_kr560_r3100_2_robot" params="prefix package_name *origin">
+  <xacro:macro name="kuka_kr560_r3100_2_robot" params="prefix package_name parent_link *origin">
     <!-- links - main serial chain -->
-    <link name="world"/>
     <link name="${prefix}base_link">
       <collision>
@@ -138,5 +137,5 @@
     </link>
     <joint name="${prefix}world-base_link" type="fixed">
-      <parent link="world"/>
+      <parent link="${parent_link}"/>
       <child link="${prefix}base_link"/>
       <xacro:insert_block name="origin"/>

Commit message: move fixed joint out of macro
also remove `parent_link` and `origin` block, better fix to #103

File: kuka_fortec_support/urdf/kr560_r3100_2_macro.xacro (robot description, xacro)
@@ -1,5 +1,5 @@
 <?xml version="1.0"?>
 <robot xmlns:xacro="http://wiki.ros.org/xacro">
-  <xacro:macro name="kuka_kr560_r3100_2_robot" params="prefix package_name parent_link *origin">
+  <xacro:macro name="kuka_kr560_r3100_2_robot" params="prefix package_name">
     <!-- links - main serial chain -->
     <link name="${prefix}base_link">
@@ -136,9 +136,4 @@
       </visual>
     </link>
-    <joint name="${prefix}world-base_link" type="fixed">
-      <parent link="${parent_link}"/>
-      <child link="${prefix}base_link"/>
-      <xacro:insert_block name="origin"/>
-    </joint>
     <joint name="${prefix}joint_1" type="revolute">
       <axis xyz="0.0 0.0 1.0"/>
