Commit message: fix to local urdf launch to make it work with temp changes
this is a follow up change to fix #103

File: kuka_fortec_support/urdf/kr560_r3100_2.urdf.xacro (robot description, xacro)
@@ -20,6 +20,7 @@
   <xacro:arg name="pitch" default="0"/>
   <xacro:arg name="yaw" default="0"/>
+  <link name="world"/>
   <xacro:kuka_fortec_ros2_control name="$(arg prefix)kr560_r3100_2" driver_version="$(arg driver_version)" client_ip="$(arg client_ip)" client_port="$(arg client_port)" controller_ip="$(arg controller_ip)" prefix="$(arg prefix)" mode="$(arg mode)" use_gpio="$(arg use_gpio)" roundtrip_time="$(arg roundtrip_time)" verify_robot_model="$(arg verify_robot_model)"/>
-  <xacro:kuka_kr560_r3100_2_robot prefix="$(arg prefix)" package_name="kuka_fortec_support">
+  <xacro:kuka_kr560_r3100_2_robot prefix="$(arg prefix)" package_name="kuka_fortec_support" parent_link="world">
     <origin xyz="$(arg x) $(arg y) $(arg z)" rpy="$(arg roll) $(arg pitch) $(arg yaw)"/>
   </xacro:kuka_kr560_r3100_2_robot>

Commit message: move fixed joint in main urdf from macro
also remove `parent_link` and `origin` block, to finish fix to kroshu#103

File: kuka_fortec_support/urdf/kr560_r3100_2.urdf.xacro (robot description, xacro)
@@ -20,8 +20,14 @@
   <xacro:arg name="pitch" default="0"/>
   <xacro:arg name="yaw" default="0"/>
+  <!-- Link list -->
   <link name="world"/>
+  <!-- Joint list -->
+  <joint name="world-base_link" type="fixed">
+    <parent link="world"/>
+    <child link="$(arg prefix)base_link"/>
+    <origin rpy="0.0 0.0 0.0" xyz="0.0 0.0 0.0"/>
+  </joint>
+  <!-- Macro instances  -->
   <xacro:kuka_fortec_ros2_control name="$(arg prefix)kr560_r3100_2" driver_version="$(arg driver_version)" client_ip="$(arg client_ip)" client_port="$(arg client_port)" controller_ip="$(arg controller_ip)" prefix="$(arg prefix)" mode="$(arg mode)" use_gpio="$(arg use_gpio)" roundtrip_time="$(arg roundtrip_time)" verify_robot_model="$(arg verify_robot_model)"/>
-  <xacro:kuka_kr560_r3100_2_robot prefix="$(arg prefix)" package_name="kuka_fortec_support" parent_link="world">
-    <origin xyz="$(arg x) $(arg y) $(arg z)" rpy="$(arg roll) $(arg pitch) $(arg yaw)"/>
-  </xacro:kuka_kr560_r3100_2_robot>
+  <xacro:kuka_kr560_r3100_2_robot prefix="$(arg prefix)" package_name="kuka_fortec_support"/>
 </robot>
